Commit message: removing engine collisions

File: src/tito_bringup/urdf/tito.urdf (robot description, URDF)
Before this commit: robot tito_robot, 14 links, 13 joints
Links:
- link engine1: geometry visual mesh filename=file:///home/benjamin/tito_ws/src/tito_bringup/meshes/engin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
- link engine2: geometry visual mesh filename=file:///home/benjamin/tito_ws/src/tito_bringup/meshes/engin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
- link engine3: geometry visual mesh filename=file:///home/benjamin/tito_ws/src/tito_bringup/meshes/engin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
- link engine4: geometry visual mesh filename=file:///home/benjamin/tito_ws/src/tito_bringup/meshes/engin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
- link engine5: geometry visual mesh filename=file:///home/benjamin/tito_ws/src/tito_bringup/meshes/engin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
- link engine6: geometry visual mesh filename=file:///home/benjamin/tito_ws/src/tito_bringup/meshes/engin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
