Commit message: simulation working with diff drive plugin

File: install/tito_bringup/share/tito_bringup/urdf/tito.urdf (robot description, URDF)
Before this commit: robot tito_robot, 14 links, 13 joints
Links:
- removed link base_link
- link engine1: geometry visual mesh filename=file:///home/benjamin/tito_ws/src/tito_bringup/meshes/engin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
- link engine2: geometry visual mesh filename=file:///home/benjamin/tito_ws/src/tito_bringup/meshes/engin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
- link engine3: geometry visual mesh filename=file:///home/benjamin/tito_ws/src/tito_bringup/meshes/engin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
- link engine4: geometry visual mesh filename=file:///home/benjamin/tito_ws/src/tito_bringup/meshes/engin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
- link engine5: geometry visual mesh filename=file:///home/benjamin/tito_ws/src/tito_bringup/meshes/engin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
- link engine6: geometry visual mesh filename=file:///home/benjamin/tito_ws/src/tito_bringup/meshes/engin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
Joints:
- removed joint base_link_joint

File: src/tito_bringup/urdf/tito.urdf (robot description, URDF)
Before this commit: robot tito_robot, 14 links, 13 joints
Links:
- removed link base_link
Joints:
- removed joint base_link_joint

Commit message: velocity controller with mimic joints working in ignition

File: install/tito_bringup/share/tito_bringup/urdf/tito.urdf (robot description, URDF)
Before this commit: robot tito_robot, 13 links, 12 joints
Joints:
- joint leg1_joint: limit lower=0 upper=0 effort=0 velocity=0 -> lower=-15 upper=15 effort=1000.0 velocity=30
- joint leg2_joint: limit lower=0 upper=0 effort=0 velocity=0 -> lower=-15 upper=15 effort=1000.0 velocity=30
- joint leg3_joint: limit lower=0 upper=0 effort=0 velocity=0 -> lower=-15 upper=15 effort=1000.0 velocity=30
- joint leg4_joint: limit lower=0 upper=0 effort=0 velocity=0 -> lower=-15 upper=15 effort=1000.0 velocity=30
- joint leg5_joint: limit lower=0 upper=0 effort=0 velocity=0 -> lower=-15 upper=15 effort=1000.0 velocity=30
- joint leg6_joint: limit lower=0 upper=0 effort=0 velocity=0 -> lower=-15 upper=15 effort=1000.0 velocity=30

Commit message: cleaning code and fitting leg 2

File: install/tito_bringup/share/tito_bringup/urdf/tito.urdf (robot description, URDF)
Before this commit: robot tito_robot, 13 links, 12 joints
Joints:
- joint leg2_joint: origin xyz=-0.10151 0 0 rpy=0 -1.5708 0 -> xyz=-0.10151 0 0 rpy=0 -1.5708 3.1416
- joint leg4_joint: origin xyz=-0.0855123716995091 0 0 rpy=3.14159265358979 -1.5707963267949 0 -> xyz=-0.1855123716995091 0 0 rpy=3.14159265358979 -1.5707963267949 3.1416

File: src/tito_bringup/urdf/tito.urdf (robot description, URDF)
Before this commit: robot tito_robot, 13 links, 12 joints
Joints:
- joint leg2_joint: origin xyz=-0.10151 0 0 rpy=0 -1.5708 0 -> xyz=-0.10151 0 0 rpy=0 -1.5708 3.1416
- joint leg4_joint: origin xyz=-0.0855123716995091 0 0 rpy=3.14159265358979 -1.5707963267949 0 -> xyz=-0.0855123716995091 0 0 rpy=3.14159265358979 -1.5707963267949 3.1416

Commit message: tito walking

File: install/tito_bringup/share/tito_bringup/urdf/tito.urdf (robot description, URDF)
Before this commit: robot tito_robot, 13 links, 12 joints
Joints:
- joint leg2_joint: origin xyz=-0.10151 0 0 rpy=0 -1.5708 3.1416 -> xyz=-0.10151 0 0 rpy=0 1.57 3.14
- joint leg4_joint: origin xyz=-0.1855123716995091 0 0 rpy=3.14159265358979 -1.5707963267949 3.1416 -> xyz=-0.0855123716995093 0 0 rpy=0 1.57 0
- joint leg6_joint: origin xyz=-0.0855123716995156 0 0 rpy=3.14159265358979 -1.5707963267949 0 -> xyz=-0.0855123716995093 0 0 rpy=0 1.57 0

File: src/tito_bringup/urdf/tito.urdf (robot description, URDF)
Before this commit: robot tito_robot, 13 links, 12 joints
Joints:
- joint leg2_joint: origin xyz=-0.10151 0 0 rpy=0 -1.5708 3.1416 -> xyz=-0.10151 0 0 rpy=0 1.57 3.14
- joint leg4_joint: origin xyz=-0.0855123716995091 0 0 rpy=3.14159265358979 -1.5707963267949 3.1416 -> xyz=-0.0855123716995093 0 0 rpy=0 1.57 0
- joint leg6_joint: origin xyz=-0.0855123716995156 0 0 rpy=3.14159265358979 -1.5707963267949 0 -> xyz=-0.0855123716995093 0 0 rpy=0 1.57 0

Commit message: foward control working

File: install/tito_bringup/share/tito_bringup/urdf/tito.urdf (robot description, URDF)
Before this commit: robot tito_robot, 13 links, 12 joints
Joints:
- joint leg4_joint: mimic joint=leg1_joint -> joint=leg2_joint
- joint leg6_joint: mimic joint=leg1_joint -> joint=leg2_joint
